File: Solder.kicad_pcb (KiCad board)
At the start: 2 copper layers, 139.2 x 94 mm, 78 parts, among them K1 SRD-24VDC-SL-C, X1 НАГРЕВ, X10 ПИТАНИЕ, X11 КОРПУС, X2 ТОКОСЪЁМ, X3 ТЕРМО, X4 ВИБРО, X5 1x01, X6 1x01, X7 1x01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

Commit message: Fixed board captions
Parts:
- moved C10 46.4 mm to (147.6, 118.9)
- moved C14 46.4 mm to (199.1, 111.8)
- moved C15 46.4 mm to (182.1, 132.7)
- moved DA1 46.4 mm to (199.6, 99.1)
- moved DA3 46.4 mm to (164.6, 70.1)
- moved DD1 46.4 mm to (127.3, 54.1)
- moved R10 46.4 mm to (176.8, 121.4)
- moved R13 46.4 mm to (183.2, 111.3)
- moved R15 46.4 mm to (149.5, 101.1)
- moved R17 46.4 mm to (177.5, 64.3)
- moved R19 46.4 mm to (162.9, 106.2)
- moved R3 46.4 mm to (131.8, 114.8)
- moved R4 46.4 mm to (164.8, 124.6)
- moved R6 46.4 mm to (136.4, 110.2)
- moved R7 46.4 mm to (148.8, 84.6)
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